File: ECAD/Garage_Controller.brd (EAGLE design)
At the start: 127 x 92.7 mm, 93 parts, among them IC1 LM358D, IC2 LM358D, J1 1885410000, J2 1885410000, J3 1885430000, J4 1885430000, J5 1885430000, J6 1885430000, J7 1885430000, Q1 35A/25V/8.5mΩ, Q2 35A/25V/8.5mΩ, Q3 35A/25V/8.5mΩ, Q4 35A/25V/8.5mΩ, U1 MCP4728-E/UN, U2 +5V, U3 +5V, U4 +3V3, U5 PCF8574ADWR

Commit message: Ordered PWBs
Parts:
- removed LED7, LED8: (no value), led:CHIP-LED0805
- removed OK2: HCPL2730, optocoupler:DIL08
- removed R16, R18: 1k, resistor:R0805
- removed R17: 3.3k, resistor:R0805
- removed R21, R22: 150, resistor:R0805
- added U6: P82B715DR, texas:SO-08
- added U7: +5V, SparkFun-IC-Power:TO-252
- R14, R15: value 3.3k -> 1k
- moved C2 18.0 mm to (78.1, 37.5), turned to 90 degrees
- moved R14 8.84 mm to (73.7, 30.5), turned to 90 degrees
- moved R15 3.24 mm to (71.1, 30.5), turned to 90 degrees
Connections:
- removed net DI2: LED7.C, OK2.7, R15.1, U5.11
- removed net DI3: LED8.C, OK2.6, R17.1, U5.12
- removed net N$22: J5.7, J5.8, R18.2
- removed net N$23: OK2.3, R18.1
- removed net N$28: LED7.A, R21.1
- removed net N$30: LED8.A, R22.1
- net +3V3: no longer C2.1, R14.2, R15.2, R17.2, R21.2, R22.2
- net +5V/1: now also J5.7, J5.8, U6.8, U7.1; no longer J5.5, J5.6, OK2.1, OK2.4
- net GND: now also C2.2, U6.4, U7.3; no longer OK2.5
- net N$20: now also J5.5, J5.6, R14.1, U6.2; no longer OK2.2, R16.1
- net N$21: now also C2.1, R14.2, R15.2, U7.2; no longer C2.2, OK2.8, R14.1
- net N$25: now also R15.1, U6.7; no longer R16.2
- net SCL: now also U6.6
- net SDA: now also U6.3
Routing:
- net SDA: track 80.2 -> 141.4 mm
- net DI3: track 57.0 -> 0.00 mm
- net SCL: track 83.2 -> 138.2 mm
- net DI2: track 53.0 -> 0.00 mm
- net +3V3: track 172.6 -> 131.1 mm, vias 6 -> 5
- net N$20: track 5.18 -> 29.0 mm
- net +5V/1: track 123.2 -> 144.7 mm, vias 3 -> 4
- net N$25: track 12.3 -> 29.0 mm
- net N$22: track 12.3 -> 0.00 mm
- net N$23: track 5.18 -> 0.00 mm
- net N$21: track 8.02 -> 12.8 mm, vias 0 -> 2
- net N$28: track 2.89 -> 0.00 mm
- net N$30: track 2.89 -> 0.00 mm
Other:
- board text added: "SCL"
- board text added: "SDA"
