File: ECAD/Garage_Controller.sch (EAGLE design)
At the start: 93 parts, among them IC1 LM358D, IC2 LM358D, J1 1885410000, J2 1885410000, J3 1885430000, J4 1885430000, J5 1885430000, J6 1885430000, J7 1885430000, Q1 35A/25V/8.5mΩ, Q2 35A/25V/8.5mΩ, Q3 35A/25V/8.5mΩ, Q4 35A/25V/8.5mΩ, U1 MCP4728-E/UN, U2 +5V, U3 +5V, U4 +3V3, U5 PCF8574ADWR

Commit message: Ordered PWBs
Parts:
- removed LED7, LED8: (no value), led:LEDCHIP-LED0805
- removed OK2: HCPL2730, optocoupler:HCPL2730
- removed R16, R18: 1k, resistor:R-US_R0805
- removed R17: 3.3k, resistor:R-US_R0805
- removed R21, R22: 150, resistor:R-US_R0805
- added U6: P82B715DR, texas:P82B715DR
- added U7: +5V, SparkFun-IC-Power:V_REG_78XX7812
- R14, R15: value 3.3k -> 1k
Connections:
- removed net DI2: LED7.C, OK2A.VO1, R15.1, U5.P6
- removed net DI3: LED8.C, OK2B.VO2, R17.1, U5.P7
- removed net N$22: J5.7, J5.8, R18.2
- removed net N$23: OK2B.C2, R18.1
- removed net N$28: LED7.A, R21.1
- removed net N$30: LED8.A, R22.1
- net +3V3: no longer C2.1, R14.2, R15.2, R17.2, R21.2, R22.2
- net +5V/1: now also J5.7, J5.8, U6.VCC, U7.IN; no longer J5.5, J5.6, OK2A.A1, OK2B.A2
- net GND: now also C2.2, U6.GND, U7.GND; no longer OK2A.GND
- net N$20: now also J5.5, J5.6, R14.1, U6.LX; no longer OK2A.C1, R16.1
- net N$21: now also C2.1, R14.2, R15.2, U7.OUT; no longer C2.2, OK2A.VCC, R14.1
- net N$25: now also R15.1, U6.LY; no longer R16.2
- net SCL: now also U6.SY
- net SDA: now also U6.SX
Other:
- moved on the sheet: C2, R14, R15
