File: ECAD/Sensor Board.brd (EAGLE design)
At the start: 38.1 x 76.2 mm, 42 parts, among them U1 +12v

Commit message: Ordered PWBs
Parts:
- added U2: P82B715DR, texas:SO-08
- moved LCL 2.54 mm to (25.4, 73.7)
- moved LDA 2.54 mm to (27.9, 73.7)
- renumbered U$1 to U3
Connections:
- new net N$11: LCL.1, U2.2
- new net N$9: LDA.1, U2.7
- net +3V3: now also U2.8
- net GND: now also U2.4
- net SCL: now also U2.3
- net SDA: now also U2.6
Routing:
- net SDA: track 0.00 -> 90.8 mm, vias 0 -> 2
- net SCL: track 0.00 -> 90.1 mm, vias 0 -> 2
- net N$11: track 0.00 -> 24.8 mm
- net N$9: track 0.00 -> 24.0 mm
- net +3V3: track 195.0 -> 197.8 mm, vias 7 -> 8
Other:
- outline, holes or cut-outs redrawn
