File: ECAD/Sensor Board.sch (EAGLE design)
At the start: 42 parts, among them U1 +12v

Commit message: Ordered PWBs
Parts:
- added U2: P82B715DR, texas:P82B715DR
- renumbered U$1 to U3
Connections:
- new net N$11: LCL.P, U2.LX
- new net N$9: LDA.P, U2.LY
- net +3V3: now also U2.VCC
- net GND: now also U2.GND
- net SCL: now also U2.SX
- net SDA: now also U2.SY
Other:
- moved on the sheet: LCL, LDA
Changed lines of the file:
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@@
 </classes>
 <parts>
-<part name="U$1" library="texas" deviceset="ADS1115" device=""/>
+<part name="U3" library="texas" deviceset="ADS1115" device=""/>
 <part name="SUPPLY1" library="supply2" deviceset="GND" device=""/>
 <part name="R1" library="resistor" deviceset="R-US_" device="R0805"/>
@@
 <part name="GND2" library="wirepad" deviceset="WIREPAD" device="SMD1,27-254" value="WIREPADSMD1,27-254"/>
 <part name="SUPPLY20" library="supply2" deviceset="GND" device=""/>
+<part name="U2" library="texas" deviceset="P82B715DR" device=""/>
+<part name="SUPPLY21" library="supply2" deviceset="GND" device=""/>
+<part name="+3V12" library="supply1" deviceset="+3V3" device=""/>
 </parts>
 <sheets>
@@
 </plain>
 <instances>
-<instance part="U$1" gate="A" x="2.54" y="35.56"/>
+<instance part="U3" gate="A" x="2.54" y="35.56"/>
 <instance part="SUPPLY1" gate="GND" x="2.54" y="17.78"/>
 <instance part="R1" gate="G$1" x="38.1" y="40.64" rot="R90"/>
@@
 <instance part="S4VCC" gate="G$1" x="-58.42" y="53.34" rot="R180"/>
 <instance part="SUPPLY10" gate="GND" x="-60.96" y="27.94"/>
-<instance part="LCL" gate="G$1" x="-7.62" y="111.76" rot="R270"/>
-<instance part="LDA" gate="G$1" x="5.08" y="111.76" rot="R270"/>
+<instance part="LCL" gate="G$1" x="-35.56" y="154.94" rot="R270"/>
+<instance part="LDA" gate="G$1" x="48.26" y="160.02" rot="R270"/>
 <instance part="S5GND" gate="G$1" x="-68.58" y="-20.32" rot="R180"/>
 <instance part="S5SDA" gate="G$1" x="-68.58" y="-12.7" rot="R180"/>
@@
 <instance part="GND2" gate="G$1" x="17.78" y="111.76" rot="R270"/>
 <instance part="SUPPLY20" gate="GND" x="17.78" y="106.68"/>
+<instance part="U2" gate="A" x="-22.86" y="152.4"/>
+<instance part="SUPPLY21" gate="GND" x="-22.86" y="142.24"/>
+<instance part="+3V12" gate="G$1" x="35.56" y="162.56"/>
 </instances>
 <busses>
@@
 <net name="GND" class="0">
 <segment>
-<pinref part="U$1" gate="A" pin="GND"/>
+<pinref part="U3" gate="A" pin="GND"/>
 <pinref part="SUPPLY1" gate="GND" pin="GND"/>
 </segment>
@@
 <pinref part="SUPPLY20" gate="GND" pin="GND"/>
 </segment>
+<segment>
+<pinref part="U2" gate="A" pin="GND"/>
+<pinref part="SUPPLY21" gate="GND" pin="GND"/>
+</segment>
 </net>
 <net name="N$1" class="0">
 <segment>
-<pinref part="U$1" gate="A" pin="ALERT"/>
+<pinref part="U3" gate="A" pin="ALERT"/>
 <pinref part="R1" gate="G$1" pin="1"/>
 <wire x1="17.78" y1="35.56" x2="38.1" y2="35.56" width="0.1524" layer="91"/>
@@
 <net name="SCL" class="0">
 <segment>
-<pinref part="U$1" gate="A" pin="SCL"/>
+<pinref part="U3" gate="A" pin="SCL"/>
 <wire x1="17.78" y1="40.64" x2="22.86" y2="40.64" width="0.1524" layer="91"/>
 <label x="22.86" y="40.64" size="1.778" layer="95"/>
@@
 <label x="-76.2" y="-5.08" size="1.778" layer="95" rot="R180"/>
 </segment>
+<segment>
+<pinref part="U2" gate="A" pin="SX"/>
+<wire x1="-22.86" y1="147.32" x2="-27.94" y2="147.32" width="0.1524" layer="91"/>
+<label x="-27.94" y="147.32" size="1.778" layer="95" rot="R180"/>
+</segment>
 </net>
 <net name="SDA" class="0">
 <segment>
-<pinref part="U$1" gate="A" pin="SDA"/>
+<pinref part="U3" gate="A" pin="SDA"/>
 <wire x1="17.78" y1="38.1" x2="22.86" y2="38.1" width="0.1524" layer="91"/>
 <label x="22.86" y="38.1" size="1.778" layer="95"/>
@@
 <label x="-76.2" y="-12.7" size="1.778" layer="95" rot="R180"/>
 </segment>
+<segment>
+<pinref part="U2" gate="A" pin="SY"/>
+<wire x1="33.02" y1="147.32" x2="38.1" y2="147.32" width="0.1524" layer="91"/>
+<label x="38.1" y="147.32" size="1.778" layer="95"/>
+</segment>
 </net>
 <net name="+3V3" class="0">
 <segment>
-<pinref part="U$1" gate="A" pin="VDD"/>
+<pinref part="U3" gate="A" pin="VDD"/>
 <pinref part="+3V1" gate="G$1" pin="+3V3"/>
 <wire x1="2.54" y1="78.74" x2="2.54" y2="66.04" width="0.1524" layer="91"/>
@@
 <pinref part="+3V11" gate="G$1" pin="+3V3"/>
 </segment>
+<segment>
+<pinref part="U2" gate="A" pin="VCC"/>
+<pinref part="+3V12" gate="G$1" pin="+3V3"/>
+<wire x1="33.02" y1="152.4" x2="35.56" y2="152.4" width="0.1524" layer="91"/>
+<wire x1="35.56" y1="152.4" x2="35.56" y2="160.02" width="0.1524" layer="91"/>
+</segment>
 </net>
 <net name="A0" class="0">
@@
 </segment>
 <segment>
-<pinref part="U$1" gate="A" pin="AIN0"/>
+<pinref part="U3" gate="A" pin="AIN0"/>
 <wire x1="-12.7" y1="40.64" x2="-17.78" y2="40.64" width="0.1524" layer="91"/>
 <label x="-17.78" y="40.64" size="1.778" layer="95" rot="R180"/>
@@
 <net name="A1" class="0">
 <segment>
-<pinref part="U$1" gate="A" pin="AIN1"/>
+<pinref part="U3" gate="A" pin="AIN1"/>
 <wire x1="-12.7" y1="38.1" x2="-17.78" y2="38.1" width="0.1524" layer="91"/>
 <label x="-17.78" y="38.1" size="1.778" layer="95" rot="R180"/>
@@
 <net name="A2" class="0">
 <segment>
-<pinref part="U$1" gate="A" pin="AIN2"/>
+<pinref part="U3" gate="A" pin="AIN2"/>
 <wire x1="-12.7" y1="35.56" x2="-17.78" y2="35.56" width="0.1524" layer="91"/>
 <label x="-17.78" y="35.56" size="1.778" layer="95" rot="R180"/>
@@
 <net name="A3" class="0">
 <segment>
-<pinref part="U$1" gate="A" pin="AIN3"/>
+<pinref part="U3" gate="A" pin="AIN3"/>
 <wire x1="-12.7" y1="33.02" x2="-17.78" y2="33.02" width="0.1524" layer="91"/>
 <label x="-17.78" y="33.02" size="1.778" layer="95" rot="R180"/>
@@
 <net name="N$4" class="0">
 <segment>
-<pinref part="U$1" gate="A" pin="ADDR"/>
+<pinref part="U3" gate="A" pin="ADDR"/>
 <pinref part="JP3" gate="G$1" pin="2"/>
 <wire x1="17.78" y1="33.02" x2="50.8" y2="33.02" width="0.1524" layer="91"/>
@@
 </segment>
 </net>
+<net name="N$9" class="0">
+<segment>
+<pinref part="U2" gate="A" pin="LY"/>
+<pinref part="LDA" gate="G$1" pin="P"/>
+<wire x1="33.02" y1="149.86" x2="48.26" y2="149.86" width="0.1524" layer="91"/>
+<wire x1="48.26" y1="149.86" x2="48.26" y2="157.48" width="0.1524" layer="91"/>
+</segment>
+</net>
+<net name="N$11" class="0">
+<segment>
+<pinref part="U2" gate="A" pin="LX"/>
+<pinref part="LCL" gate="G$1" pin="P"/>
+<wire x1="-22.86" y1="149.86" x2="-35.56" y2="149.86" width="0.1524" layer="91"/>
+<wire x1="-35.56" y1="149.86" x2="-35.56" y2="152.4" width="0.1524" layer="91"/>
+</segment>
+</net>
